File: FinalPcbLayout/power.kicad_sch (KiCad schematic)
At the start: 33 parts, among them Q1 NMOS, U4 AMS1117-3.3

Commit message: tyra's changes
Parts:
- C1, C2, C3, C8: footprint Capacitor_SMD:C_0603_1608Metric -> Capacitor_SMD:C_0402_1005Metric
- C10, C19, C6, C9: footprint Capacitor_SMD:C_0603_1608Metric -> Capacitor_SMD:C_0805_2012Metric
- R3, R4: footprint Resistor_SMD:R_0603_1608Metric -> Resistor_SMD:R_1206_3216Metric
Changed lines of the file:
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@@
       (effects (font (size 1.27 1.27)) (justify right))
     )
-    (property "Footprint" "Capacitor_SMD:C_0603_1608Metric" (at 76.5048 63.5 0)
+    (property "Footprint" "Capacitor_SMD:C_0402_1005Metric" (at 76.5048 63.5 0)
       (effects (font (size 1.27 1.27)) hide)
     )
@@
       (effects (font (size 1.27 1.27)) (justify right))
     )
-    (property "Footprint" "Capacitor_SMD:C_0603_1608Metric" (at 94.2848 93.98 0)
+    (property "Footprint" "Capacitor_SMD:C_0402_1005Metric" (at 94.2848 93.98 0)
       (effects (font (size 1.27 1.27)) hide)
     )
@@
       (effects (font (size 1.27 1.27)) (justify right))
     )
-    (property "Footprint" "Resistor_SMD:R_0603_1608Metric" (at 197.104 92.456 90)
+    (property "Footprint" "Resistor_SMD:R_1206_3216Metric" (at 197.104 92.456 90)
       (effects (font (size 1.27 1.27)) hide)
     )
@@
       (effects (font (size 1.27 1.27)) (justify left))
     )
-    (property "Footprint" "Capacitor_SMD:C_0603_1608Metric" (at 260.0452 140.97 0)
+    (property "Footprint" "Capacitor_SMD:C_0805_2012Metric" (at 260.0452 140.97 0)
       (effects (font (size 1.27 1.27)) hide)
     )
@@
       (effects (font (size 1.27 1.27)) (justify right))
     )
-    (property "Footprint" "Capacitor_SMD:C_0603_1608Metric" (at 106.9848 93.98 0)
+    (property "Footprint" "Capacitor_SMD:C_0402_1005Metric" (at 106.9848 93.98 0)
       (effects (font (size 1.27 1.27)) hide)
     )
@@
       (effects (font (size 1.27 1.27)))
     )
-    (property "Footprint" "Resistor_SMD:R_0603_1608Metric" (at 162.306 72.136 90)
+    (property "Footprint" "Resistor_SMD:R_1206_3216Metric" (at 162.306 72.136 90)
       (effects (font (size 1.27 1.27)) hide)
     )
@@
       (effects (font (size 1.27 1.27)) (justify right))
     )
-    (property "Footprint" "Capacitor_SMD:C_0603_1608Metric" (at 171.7548 90.17 0)
+    (property "Footprint" "Capacitor_SMD:C_0805_2012Metric" (at 171.7548 90.17 0)
       (effects (font (size 1.27 1.27)) hide)
     )
@@
       (effects (font (size 1.27 1.27)) (justify right))
     )
-    (property "Footprint" "Capacitor_SMD:C_0603_1608Metric" (at 253.0348 88.9 0)
+    (property "Footprint" "Capacitor_SMD:C_0402_1005Metric" (at 253.0348 88.9 0)
       (effects (font (size 1.27 1.27)) hide)
     )
@@
       (effects (font (size 1.27 1.27)) (justify left))
     )
-    (property "Footprint" "Capacitor_SMD:C_0603_1608Metric" (at 55.5752 143.51 0)
+    (property "Footprint" "Capacitor_SMD:C_0805_2012Metric" (at 55.5752 143.51 0)
       (effects (font (size 1.27 1.27)) hide)
     )
@@
       (effects (font (size 1.27 1.27)) (justify right))
     )
-    (property "Footprint" "Capacitor_SMD:C_0603_1608Metric" (at 68.8848 82.55 0)
-      (effects (font (size 1.27 1.27)) hide)
-    )
+    (property "Footprint" "Capacitor_SMD:C_0805_2012Metric" (at 68.8848 82.55 0)
+      (effects (font (size 1.27 1.27)) hide)
+    )
