File: FinalPcbLayout/power.kicad_sch (KiCad schematic)
At the start: 42 parts, among them J3 Barrel_Jack, Q1 NMOS, Q4 PMOS, Q5 PMOS, U4 AMS1117-3.3

Commit message: Links and costs
Parts:
- C1, C17, C2: Cost 0 -> $0.26; Order-Link (none) -> https://www.digikey.com/en/products/detail/samsung-electro-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
- C10, C16, C18, C5, C8: Cost 0 -> $0.10; Order-Link (none) -> https://www.digikey.com/en/products/detail/samsung-electro-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
- C11, C7: Cost 0 -> $0.08; Order-Link (none) -> https://www.digikey.com/en/products/detail/murata-electroni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
- C19: Cost 0 -> $0.29; Order-Link (none) -> https://www.digikey.com/en/products/detail/samsung-electro-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
- C3: Cost 0 -> $0.45; Order-Link (none) -> https://www.digikey.com/en/products/detail/kemet/C0603C682K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
- C4: Cost 0 -> $0.38; Order-Link (none) -> https://www.digikey.com/en/products/detail/kemet/C0603C153J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
- C6: Cost 0 -> $0.42; Order-Link (none) -> https://www.digikey.com/en/products/detail/kemet/C0805C102K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
- C9: Cost (uuid fabb1e82-3a32-4eed-b578-540d99c03e17) -> $0.10; Order-Link (none) -> https://www.digikey.com/en/products/detail/samsung-electro-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
- L1: Cost 0 -> $0.11; Order-Link (none) -> https://www.digikey.com/en/products/detail/taiyo-yuden/LBR2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
- R1: Cost 0 -> $0.10; Order-Link (none) -> https://www.digikey.com/en/products/detail/yageo/RC0603JR-1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
- R10, R11, R12, R13, R2, R23, R24, R4: Cost 0 -> $0.10; Order-Link (none) -> https://www.digikey.com/en/products/detail/stackpole-electr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
- R25, R5, R7: Cost 0 -> $0.10; Order-Link (none) -> https://www.digikey.com/en/products/detail/yageo/RC0603FR-0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
- R3: Cost 0 -> $0.58; Order-Link (none) -> https://www.digikey.com/en/products/detail/vishay-dale/WFCP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
- R6: Cost 0 -> $0.13; Order-Link (none) -> https://www.digikey.com/en/products/detail/panasonic-electr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

Commit message: some footprint updates
Parts:
- C4: Cost $0.38 -> $0.22; Order-Link https://www.digikey.com/en/products/detail/kemet/C0603C153J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 -> https://www.digikey.com/en/products/detail/cal-chip-electro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
- R25: Order-Link https://www.digikey.com/en/products/detail/yageo/RC0603FR-0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 -> https://www.digikey.com/en/products/detail/yageo/RC0805FR-0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
- R3: Cost $0.58 -> $0.71; Order-Link https://www.digikey.com/en/products/detail/vishay-dale/WFCP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 -> https://www.digikey.com/en/products/detail/panasonic-electr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
- R4: Order-Link https://www.digikey.com/en/products/detail/stackpole-electr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 -> https://www.digikey.com/en/products/detail/koa-speer-electr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
Changed lines of the file:
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@@
       (effects (font (size 1.27 1.27)) hide)
     )
-    (property "Order-Link" "https://www.digikey.com/en/products/detail/yageo/RC0603FR-07487RL/727262" (at 271.78 147.32 0)
+    (property "Order-Link" "https://www.digikey.com/en/products/detail/yageo/RC0805FR-07100RL/727543" (at 271.78 147.32 0)
       (effects (font (size 1.27 1.27)) hide)
     )
@@
       (effects (font (size 1.27 1.27)) hide)
     )
-    (property "Cost" "$0.58" (at 218.44 78.74 0)
+    (property "Cost" "$0.71" (at 218.44 78.74 0)
       (effects (font (size 1.27 1.27)) hide)
     )
@@
       (effects (font (size 1.27 1.27)) hide)
     )
-    (property "Order-Link" "https://www.digikey.com/en/products/detail/vishay-dale/WFCP0603R0120FE66/15908415" (at 218.44 78.74 0)
+    (property "Order-Link" "https://www.digikey.com/en/products/detail/panasonic-electronic-components/ERJ-8CWFR012V/4926999" (at 218.44 78.74 0)
       (effects (font (size 1.27 1.27)) hide)
     )
@@
       (effects (font (size 1.27 1.27)) hide)
     )
-    (property "Order-Link" "https://www.digikey.com/en/products/detail/stackpole-electronics-inc/RMCF0603FT487K/1714075" (at 182.88 57.15 0)
+    (property "Order-Link" "https://www.digikey.com/en/products/detail/koa-speer-electronics-inc/RK73H2BTTD4870F/10236118" (at 182.88 57.15 0)
       (effects (font (size 1.27 1.27)) hide)
     )
@@
       (effects (font (size 1.27 1.27)) hide)
     )
-    (property "Cost" "$0.38" (at 142.24 76.2 0)
+    (property "Cost" "$0.22" (at 142.24 76.2 0)
       (effects (font (size 1.27 1.27)) hide)
     )
@@
       (effects (font (size 1.27 1.27)) hide)
     )
-    (property "Order-Link" "https://www.digikey.com/en/products/detail/kemet/C0603C153J3GAC7867/2199990" (at 142.24 76.2 0)
-      (effects (font (size 1.27 1.27)) hide)
-    )
+    (property "Order-Link" "https://www.digikey.com/en/products/detail/cal-chip-electronics-inc/CHV1812N250153KXT/13558742" (at 142.24 76.2 0)
+      (effects (font (size 1.27 1.27)) hide)
+    )
