File: FinalPcbLayout/FinalPcbLayout.kicad_sch (KiCad schematic)
At the start: 19 parts, among them J1 Conn_01x04_Pin, J3 Conn_01x11_Pin, J5 Conn_02x05_Odd_Even, J6 Conn_01x02_Pin, J8 Micro_SD_Card, SW1 SW_Push, U1 ESP32-WROOM-32

Commit message: Links and costs
Parts:
- C12, C13, C14, C15: Cost 0 -> $0.10; Order-Link (none) -> https://www.digikey.com/en/products/detail/samsung-electro-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
- R8: Cost 0 -> $0.20; Order-Link (none) -> https://www.digikey.com/en/products/detail/koa-speer-electr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
Changed lines of the file:
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@@
       (effects (font (size 1.27 1.27)) hide)
     )
-    (property "Cost" "0" (at 163.83 139.7 0)
+    (property "Cost" "$0.10" (at 163.83 139.7 0)
       (effects (font (size 1.27 1.27)) hide)
     )
     (property "Sim.Enable" "0" (at 163.83 139.7 0)
+      (effects (font (size 1.27 1.27)) hide)
+    )
+    (property "Order-Link" "https://www.digikey.com/en/products/detail/samsung-electro-mechanics/CL10C221JB8NNNC/3886706" (at 163.83 139.7 0)
       (effects (font (size 1.27 1.27)) hide)
     )
@@
       (effects (font (size 1.27 1.27)) hide)
     )
-    (property "Cost" "0" (at 175.26 139.7 0)
+    (property "Cost" "$0.10" (at 175.26 139.7 0)
       (effects (font (size 1.27 1.27)) hide)
     )
     (property "Sim.Enable" "0" (at 175.26 139.7 0)
+      (effects (font (size 1.27 1.27)) hide)
+    )
+    (property "Order-Link" "https://www.digikey.com/en/products/detail/samsung-electro-mechanics/CL10C221JB8NNNC/3886706" (at 175.26 139.7 0)
       (effects (font (size 1.27 1.27)) hide)
     )
@@
       (effects (font (size 1.27 1.27)) hide)
     )
-    (property "Cost" "0" (at 102.87 148.59 0)
+    (property "Cost" "$0.10" (at 102.87 148.59 0)
       (effects (font (size 1.27 1.27)) hide)
     )
@@
       (effects (font (size 1.27 1.27)) hide)
     )
+    (property "Order-Link" "https://www.digikey.com/en/products/detail/samsung-electro-mechanics/CL21A106KOQNNNE/3886754" (at 102.87 148.59 0)
+      (effects (font (size 1.27 1.27)) hide)
+    )
     (pin "1")
     (pin "2")
@@
       (effects (font (size 1.27 1.27)) hide)
     )
-    (property "Cost" "0" (at 109.22 118.11 0)
+    (property "Cost" "$0.20" (at 109.22 118.11 0)
       (effects (font (size 1.27 1.27)) hide)
     )
     (property "Sim.Enable" "0" (at 109.22 118.11 0)
+      (effects (font (size 1.27 1.27)) hide)
+    )
+    (property "Order-Link" "https://www.digikey.com/en/products/detail/koa-speer-electronics-inc/RN73H1JTTD3703F100/10687650" (at 109.22 118.11 0)
       (effects (font (size 1.27 1.27)) hide)
     )
@@
       (effects (font (size 1.27 1.27)) hide)
     )
-    (property "Cost" "0" (at 110.49 148.59 0)
+    (property "Cost" "$0.10" (at 110.49 148.59 0)
       (effects (font (size 1.27 1.27)) hide)
     )
@@
       (effects (font (size 1.27 1.27)) hide)
     )
+    (property "Order-Link" "https://www.digikey.com/en/products/detail/samsung-electro-mechanics/CL10B104KB8NNWC/3887593" (at 110.49 148.59 0)
+      (effects (font (size 1.27 1.27)) hide)
+    )
