File: FinalPcbLayout/usb.kicad_sch (KiCad schematic)
At the start: 26 parts, among them J5 USB_C_Receptacle, Q2 NPN, Q3 NPN, U7 93LCxxB, Y1 12Mhz

Commit message: Links and costs
Parts:
- C20: Cost 0 -> $0.27; Order-Link (none) -> https://www.digikey.com/en/products/detail/tdk-corporation/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
- C21, C22: Cost 0 -> $0.10; Order-Link (none) -> https://www.digikey.com/en/products/detail/walsin-technolog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
- C23, C24: Cost 0 -> $0.10; Order-Link (none) -> https://www.digikey.com/en/products/detail/samsung-electro-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
- D2, D3: Cost 0 -> (none)
- R14, R15, R16, R17, R19, R20, R26, R27, R28, R9: Cost 0 -> $0.10; Order-Link (none) -> https://www.digikey.com/en/products/detail/stackpole-electr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
- R21: Cost 0 -> $0.13; Order-Link (none) -> https://www.digikey.com/en/products/detail/panasonic-electr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
- R22: Cost 0 -> $0.10; Order-Link (none) -> https://www.digikey.com/en/products/detail/panasonic-electr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
Changed lines of the file:
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@@
       (effects (font (size 1.27 1.27)) hide)
     )
-    (property "Cost" "0" (at 48.26 127 0)
+    (property "Cost" "$0.10" (at 48.26 127 0)
       (effects (font (size 1.27 1.27)) hide)
     )
@@
       (effects (font (size 1.27 1.27)) hide)
     )
+    (property "Order-Link" "https://www.digikey.com/en/products/detail/walsin-technology-corporation/0603N180J500CT/9354991" (at 48.26 127 0)
+      (effects (font (size 1.27 1.27)) hide)
+    )
     (pin "1")
     (pin "2")
@@
       (effects (font (size 1.27 1.27)) hide)
     )
-    (property "Cost" "0" (at 74.93 105.41 0)
+    (property "Cost" "$0.10" (at 74.93 105.41 0)
       (effects (font (size 1.27 1.27)) hide)
     )
@@
       (effects (font (size 1.27 1.27)) hide)
     )
+    (property "Order-Link" "https://www.digikey.com/en/products/detail/stackpole-electronics-inc/RMCF0603FT10K0/1761235" (at 74.93 105.41 0)
+      (effects (font (size 1.27 1.27)) hide)
+    )
     (pin "1")
     (pin "2")
@@
       (effects (font (size 1.27 1.27)) hide)
     )
-    (property "Cost" "0" (at 59.69 110.49 0)
+    (property "Cost" "$0.10" (at 59.69 110.49 0)
       (effects (font (size 1.27 1.27)) hide)
     )
@@
       (effects (font (size 1.27 1.27)) hide)
     )
+    (property "Order-Link" "https://www.digikey.com/en/products/detail/stackpole-electronics-inc/RMCF0603FT10K0/1761235" (at 59.69 110.49 0)
+      (effects (font (size 1.27 1.27)) hide)
+    )
     (pin "1")
     (pin "2")
@@
       (effects (font (size 1.27 1.27)) hide)
     )
-    (property "Cost" "0" (at 95.25 35.56 0)
+    (property "Cost" "$0.10" (at 95.25 35.56 0)
       (effects (font (size 1.27 1.27)) hide)
     )
@@
       (effects (font (size 1.27 1.27)) hide)
     )
+    (property "Order-Link" "https://www.digikey.com/en/products/detail/samsung-electro-mechanics/CL10B333KB8NNNC/3887699" (at 95.25 35.56 0)
+      (effects (font (size 1.27 1.27)) hide)
+    )
     (pin "1")
     (pin "2")
@@
       (effects (font (size 1.27 1.27)) hide)
     )
-    (property "Cost" "0" (at 48.26 137.16 0)
+    (property "Cost" "$0.10" (at 48.26 137.16 0)
       (effects (font (size 1.27 1.27)) hide)
     )
     (property "Sim.Enable" "0" (at 48.26 137.16 0)
+      (effects (font (size 1.27 1.27)) hide)
+    )
+    (property "Order-Link" "https://www.digikey.com/en/products/detail/walsin-technology-corporation/0603N180J500CT/9354991" (at 48.26 137.16 0)
       (effects (font (size 1.27 1.27)) hide)
     )
@@
       (effects (font (size 1.27 1.27)) hide)
     )
-    (property "Cost" "0" (at 149.86 143.51 0)
+    (property "Cost" "" (at 149.86 143.51 0)
       (effects (font (size 1.27 1.27)) hide)
     )
@@
       (effects (font (size 1.27 1.27)) hide)
     )
-    (property "Cost" "0" (at 139.7 177.8 0)
+    (property "Cost" "$0.10" (at 139.7 177.8 0)
       (effects (font (size 1.27 1.27)) hide)
     )
     (property "Sim.Enable" "0" (at 139.7 177.8 0)
+      (effects (font (size 1.27 1.27)) hide)
+    )
+    (property "Order-Link" "https://www.digikey.com/en/products/detail/stackpole-electronics-inc/RMCF0603FT1K00/1761077" (at 139.7 177.8 0)
       (effects (font (size 1.27 1.27)) hide)
     )
@@
       (effects (font (size 1.27 1.27)) hide)
     )
-    (property "Cost" "0" (at 83.82 35.56 0)
+    (property "Cost" "$0.13" (at 83.82 35.56 0)
       (effects (font (size 1.27 1.27)) hide)
     )
     (property "Sim.Enable" "0" (at 83.82 35.56 0)
+      (effects (font (size 1.27 1.27)) hide)
+    )
+    (property "Order-Link" "https://www.digikey.com/en/products/detail/panasonic-electronic-components/ERA-3AEB153V/1465882" (at 83.82 35.56 0)
       (effects (font (size 1.27 1.27)) hide)
     )
@@
       (effects (font (size 1.27 1.27)) hide)
     )
-    (property "Cost" "0" (at 254 45.72 0)
+    (property "Cost" "$0.10" (at 254 45.72 0)
       (effects (font (size 1.27 1.27)) hide)
     )
@@
       (effects (font (size 1.27 1.27)) hide)
     )
+    (property "Order-Link" "https://www.digikey.com/en/products/detail/panasonic-electronic-components/ERJ-3EKF2001V/196183" (at 254 45.72 0)
+      (effects (font (size 1.27 1.27)) hide)
+    )
     (pin "1")
     (pin "2")
@@
       (effects (font (size 1.27 1.27)) hide)
     )
-    (property "Cost" "0" (at 149.86 132.08 0)
+    (property "Cost" "$0.10" (at 149.86 132.08 0)
       (effects (font (size 1.27 1.27)) hide)
     )
     (property "Sim.Enable" "0" (at 149.86 132.08 0)
+      (effects (font (size 1.27 1.27)) hide)
+    )
+    (property "Order-Link" "https://www.digikey.com/en/products/detail/stackpole-electronics-inc/RMCF0603FT43R0/1714038" (at 149.86 132.08 0)
       (effects (font (size 1.27 1.27)) hide)
     )
@@
       (effects (font (size 1.27 1.27)) hide)
     )
-    (property "Cost" "0" (at 67.31 107.95 0)
+    (property "Cost" "$0.10" (at 67.31 107.95 0)
       (effects (font (size 1.27 1.27)) hide)
     )
     (property "Sim.Enable" "0" (at 67.31 107.95 0)
+      (effects (font (size 1.27 1.27)) hide)
+    )
+    (property "Order-Link" "https://www.digikey.com/en/products/detail/stackpole-electronics-inc/RMCF0603FT10K0/1761235" (at 67.31 107.95 0)
       (effects (font (size 1.27 1.27)) hide)
     )
@@
       (effects (font (size 1.27 1.27)) hide)
     )
-    (property "Cost" "0" (at 72.39 152.4 0)
+    (property "Cost" "$0.27" (at 72.39 152.4 0)
       (effects (font (size 1.27 1.27)) hide)
     )
@@
       (effects (font (size 1.27 1.27)) hide)
     )
+    (property "Order-Link" "https://www.digikey.com/en/products/detail/tdk-corporation/C1608X5R1C335K080AC/2732911" (at 72.39 152.4 0)
+      (effects (font (size 1.27 1.27)) hide)
+    )
     (pin "1")
     (pin "2")
@@
       (effects (font (size 1.27 1.27)) hide)
     )
-    (property "Cost" "0" (at 226.06 116.84 0)
+    (property "Cost" "$0.10" (at 226.06 116.84 0)
       (effects (font (size 1.27 1.27)) hide)
     )
@@
       (effects (font (size 1.27 1.27)) hide)
     )
+    (property "Order-Link" "https://www.digikey.com/en/products/detail/stackpole-electronics-inc/RMCF0603FT10K0/1761235" (at 226.06 116.84 0)
+      (effects (font (size 1.27 1.27)) hide)
+    )
     (pin "1")
     (pin "2")
@@
       (effects (font (size 1.27 1.27)) hide)
     )
-    (property "Cost" "0" (at 226.06 142.24 0)
+    (property "Cost" "$0.10" (at 226.06 142.24 0)
       (effects (font (size 1.27 1.27)) hide)
     )
     (property "Sim.Enable" "0" (at 226.06 142.24 0)
+      (effects (font (size 1.27 1.27)) hide)
+    )
+    (property "Order-Link" "https://www.digikey.com/en/products/detail/stackpole-electronics-inc/RMCF0603FT10K0/1761235" (at 226.06 142.24 0)
       (effects (font (size 1.27 1.27)) hide)
     )
@@
       (effects (font (size 1.27 1.27)) hide)
     )
-    (property "Cost" "0" (at 139.7 143.51 0)
+    (property "Cost" "" (at 139.7 143.51 0)
       (effects (font (size 1.27 1.27)) hide)
     )
@@
       (effects (font (size 1.27 1.27)) hide)
     )
-    (property "Cost" "0" (at 139.7 175.26 0)
+    (property "Cost" "$0.10" (at 139.7 175.26 0)
       (effects (font (size 1.27 1.27)) hide)
     )
@@
       (effects (font (size 1.27 1.27)) hide)
     )
+    (property "Order-Link" "https://www.digikey.com/en/products/detail/stackpole-electronics-inc/RMCF0603FT1K00/1761077" (at 139.7 175.26 0)
+      (effects (font (size 1.27 1.27)) hide)
+    )
     (pin "1")
     (pin "2")
@@
       (effects (font (size 1.27 1.27)) hide)
     )
-    (property "Cost" "0" (at 83.82 25.4 0)
+    (property "Cost" "$0.10" (at 83.82 25.4 0)
       (effects (font (size 1.27 1.27)) hide)
     )
@@
       (effects (font (size 1.27 1.27)) hide)
     )
+    (property "Order-Link" "https://www.digikey.com/en/products/detail/stackpole-electronics-inc/RMCF0603FT100K/1761112" (at 83.82 25.4 0)
+      (effects (font (size 1.27 1.27)) hide)
+    )
     (pin "1")
     (pin "2")
@@
       (effects (font (size 1.27 1.27)) hide)
     )
-    (property "Cost" "0" (at 227.33 33.02 0)
+    (property "Cost" "$0.10" (at 227.33 33.02 0)
       (effects (font (size 1.27 1.27)) hide)
     )
@@
       (effects (font (size 1.27 1.27)) hide)
     )
+    (property "Order-Link" "https://www.digikey.com/en/products/detail/samsung-electro-mechanics/CL10B104KB8NNWC/3887593" (at 227.33 33.02 0)
+      (effects (font (size 1.27 1.27)) hide)
+    )
     (pin "1")
     (pin "2")
@@
       (effects (font (size 1.27 1.27)) hide)
     )
-    (property "Cost" "0" (at 66.04 128.27 0)
+    (property "Cost" "$0.10" (at 66.04 128.27 0)
       (effects (font (size 1.27 1.27)) hide)
     )
@@
       (effects (font (size 1.27 1.27)) hide)
     )
+    (property "Order-Link" "https://www.digikey.com/en/products/detail/stackpole-electronics-inc/RMCF0603FT12K0/1761297" (at 66.04 128.27 0)
+      (effects (font (size 1.27 1.27)) hide)
+    )
