File: FinalPcbLayout/FinalPcbLayout.kicad_pcb (KiCad board)
At the start: 4 copper layers, 100.9 x 47.2 mm, 85 parts, among them J1 Conn_02x05_Odd_Even, J2 SPI, J3 Barrel_Jack, J4 C1, J5 USB_C_Receptacle, J6 Conn_01x02_Pin, J7 Display Socket, J8 Micro_SD_Card, Q1 NMOS, Q2 S8050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

Commit message: routing
Parts:
- removed C20: 3.3u, Capacitor_SMD:C_0603_1608Metric
- removed C21, C22: 18pf, Capacitor_SMD:C_0603_1608Metric
- removed C23: 33nF, Capacitor_SMD:C_0603_1608Metric
- removed C24: .1u, Capacitor_SMD:C_0603_1608Metric
- removed D2: BLUE, LED_SMD:LED_0603_1608Metric
- removed D3, D7: RED, LED_SMD:LED_0603_1608Metric
- removed FB2: FerriteBead, Resistor_SMD:R_0603_1608Metric
- removed J1: Conn_02x05_Odd_Even, Connector_PinHeader_1.27mm:PinHeader_2x05_P1.27mm_Vertical
- removed J2: SPI, TerminalBlock_TE-Connectivity:TerminalBlock_TE_282834-3_1x03_P2.54mm_Horizontal
- removed J3: Barrel_Jack, Connector_BarrelJack:BarrelJack_GCT_DCJ200-10-A_Horizontal
- removed J4: C1, TerminalBlock_TE-Connectivity:TerminalBlock_TE_282834-3_1x03_P2.54mm_Horizontal
- removed J5: USB_C_Receptacle, Connector_USB:USB_C_Receptacle_Molex_105450-0101
- removed Q2, Q3: S8050, Package_TO_SOT_THT:TO-92_Inline
- removed Q4, Q5: PMOS, Package_TO_SOT_SMD:Vishay_PowerPAK_SC70-6L_Single
- removed R14, R15: 10k 1%, Resistor_SMD:R_0603_1608Metric
- removed R16, R17: 1k, Resistor_SMD:R_0603_1608Metric
- removed R18: 25, Resistor_SMD:R_0603_1608Metric
- removed R19: 65, Resistor_SMD:R_0603_1608Metric
- removed R20: 100k 1%, Resistor_SMD:R_0603_1608Metric
- removed R21: 15k 1%, Resistor_SMD:R_0603_1608Metric
- removed R22: 2k, Resistor_SMD:R_0603_1608Metric
- removed R25: 100, Resistor_SMD:R_0805_2012Metric
- removed R26, R27, R28, R29: 10k, Resistor_SMD:R_0603_1608Metric
- removed R9: 12k 1%, Resistor_SMD:R_0603_1608Metric
- removed U6: ~, Package_DFN_QFN:QFN-56-1EP_8x8mm_P0.5mm_EP4.5x5.2mm_ThermalVias
- removed U7: 93LCxxB, Package_SO:SOIC-8_3.9x4.9mm_P1.27mm
- removed Y1: 12Mhz, Crystal:Crystal_SMD_SeikoEpson_FA238-4Pin_3.2x2.5mm
- moved U1 21.9 mm to (174.6, 102.2), turned to -90 degrees
- moved H1 2.97 mm to (83.6, 81.5)
- moved H2 2.56 mm to (83.8, 123.2)
- moved H3 1.22 mm to (179.0, 81.8)
- moved FB1 0.54 mm to (151.1, 111.5)
- moved C12 0.40 mm to (148.7, 101.4)
- moved H4 0.32 mm to (178.6, 122.5)
- moved R8 0.26 mm to (149.8, 98.8)
Connections:
- C7 pad 2: +12V -> /Power/V_in
- C8 pad 2: +12V -> /Power/V_in
- D1 pad 1: +12V -> /Power/V_in
- J7 pad 11: /Touch_CS -> /Power/V_in
- R7 pad 2: +12V -> /Power/V_in
- U1 pad 29: /Touch_CS -> /Power/V_in
Routing:
- net /SCLK: track 254.6 -> 130.4 mm, vias 3 -> 2
- net /CIPO: track 12.4 -> 135.2 mm, vias 0 -> 1
- net /Power/V_in: track 51.3 -> 172.6 mm, vias 0 -> 5
- net unconnected-(J7-Pin_9-Pad9): track 101.1 -> 0.00 mm, vias 2 -> 0
- net +3.3V: track 232.4 -> 159.0 mm, vias 2 -> 4
- net +12V: track 40.5 -> 0.00 mm, vias 2 -> 0
- net /COPI: track 112.7 -> 137.8 mm, vias 3 -> 1
- net /SD_CS: track 0.00 -> 23.4 mm
- net GND: track 53.2 -> 41.3 mm, vias 36 -> 35
- net /Display_RST: track 100.9 -> 89.4 mm, vias 2 -> 1
- net /Display_CS: track 97.3 -> 104.5 mm, vias 2 -> 1
- net Net-(U2-OUTN): track 6.75 -> 0.00 mm
- net Net-(J6-Pin_1): track 9.04 -> 2.46 mm
- net /Display_DC: track 101.0 -> 94.5 mm
- net /usb/RXLED: track 4.66 -> 0.00 mm
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Other:
- board size 100.9 x 47.2 mm -> 102.4 x 47.4 mm
